File: Sensing_Station/Sensing_Station.kicad_sch (KiCad schematic)
At the start: 29 parts, among them J1 Conn_01x02_Pin, J2 Conn_01x02_Pin, J3 Conn_01x02_Pin, Q1 2N7000, Q2 BC550, SW1 ORD 324/10-15 AT, U1 LM35CAZ/NOPB, U2 NE555P, U3 LM358

Commit message: v2.0
Connections:
- net DAQ_MAG: now also J3.2 (Pin_2); no longer J2.1 (Pin_1)
- net DAQ_SOUND: now also J3.1 (Pin_1); no longer J3.2 (Pin_2)
- net DAQ_TEMP: now also J2.1 (Pin_1); no longer J3.1 (Pin_1)
Changed lines of the file:
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@@
 		)
 	)
-	(label "DAQ_MAG"
+	(label "DAQ_TEMP"
 		(at 43.18 173.99 0)
 		(effects
@@
 		)
 	)
-	(label "DAQ_TEMP"
+	(label "DAQ_SOUND"
 		(at 43.18 184.15 0)
 		(effects
@@
 		)
 	)
-	(label "DAQ_SOUND"
+	(label "DAQ_MAG"
 		(at 43.18 186.69 0)
 		(effects

Commit message: v3.0
Parts:
- Q1: footprint Package_TO_SOT_THT:TO-92_Inline -> Package_TO_SOT_THT:TO-92_Inline_Wide
- U1: footprint SensingStation:Z03A -> Package_TO_SOT_THT:TO-92_Inline
Connections:
- net DAQ_LIGHT: now also J2.1 (Pin_1); no longer J2.2 (Pin_2)
- net DAQ_TEMP: now also J2.2 (Pin_2); no longer J2.1 (Pin_1)
Other:
- note added: "+"
Changed lines of the file:
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@@
 	(generator_version "10.0")
 	(paper "A4")
+	(text "+\n"
+		(exclude_from_sim no)
+		(at 177.038 131.318 0)
+		(effects
+			(font
+				(size 1.27 1.27)
+			)
+		)
+	)
 	(text "Magnetic Station\n"
 		(exclude_from_sim no)
@@
 		)
 	)
-	(label "DAQ_LIGHT"
+	(label "DAQ_TEMP"
 		(at 43.18 176.53 0)
 		(effects
@@
 		)
 	)
-	(label "DAQ_TEMP"
+	(label "DAQ_LIGHT"
 		(at 43.18 173.99 0)
 		(effects
@@
 			)
 		)
-		(property "Footprint" "SensingStation:Z03A"
+		(property "Footprint" "Package_TO_SOT_THT:TO-92_Inline"
 			(at 41.91 41.91 0)
 			(hide yes)
@@
 			)
 		)
-		(property "Footprint" "Package_TO_SOT_THT:TO-92_Inline"
+		(property "Footprint" "Package_TO_SOT_THT:TO-92_Inline_Wide"
 			(at 218.44 59.055 0)
 			(hide yes)
