File: Sensing_Station/Sensing_Station.kicad_pcb (KiCad board)
At the start: 2 copper layers, 50.3 x 66.3 mm, 29 parts, among them J1 Conn_01x02_Pin, J2 Conn_01x02_Pin, J3 Conn_01x02_Pin, Q1 2N7000, Q2 BC550, SW1 ORD 324/10-15 AT, U1 LM35CAZ/NOPB, U2 NE555P, U3 LM358

Commit message: v2.0
Parts:
- moved R3 48.6 mm to (118.0, 136.4), turned to 90 degrees
- moved C2 44.9 mm to (92.7, 90.3), turned to 180 degrees
- moved U3 39.1 mm to (85.1, 93.9), turned to 0 degrees
- moved R2 31.2 mm to (99.3, 99.6), turned to 90 degrees
- moved R1 27.9 mm to (95.7, 99.6), turned to 90 degrees
- moved R4 23.1 mm to (121.2, 111.6)
- moved R6 23.1 mm to (103.2, 111.1)
- moved R7 23.1 mm to (107.2, 111.1)
- moved RV1 23.1 mm to (111.5, 109.7)
- moved D1 23.1 mm to (112.3, 102.1)
- moved Q1 23.1 mm to (113.8, 96.8)
- moved R5 22.1 mm to (118.4, 97.8), turned to 0 degrees
- moved R9 16.5 mm to (91.4, 115.1)
- moved C4 16.4 mm to (104.7, 134.8)
- moved D2 16.4 mm to (99.5, 133.4)
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Connections:
- J2 pad 1: /DAQ_MAG -> /DAQ_LIGHT
- J2 pad 2: /DAQ_LIGHT -> /DAQ_TEMP
- J3 pad 1: /DAQ_TEMP -> /DAQ_SOUND
- J3 pad 2: /DAQ_SOUND -> /DAQ_MAG
Routing:
- net +5V: track 111.2 -> 92.8 mm
- net /DAQ_TEMP: track 24.1 -> 14.9 mm
- net /DAQ_LIGHT: track 31.9 -> 24.0 mm
- net Net-(Q2-B): track 18.4 -> 16.5 mm
- net /DAQ_MAG: track 9.21 -> 10.9 mm
- net /DAQ_SOUND: track 28.2 -> 26.9 mm
- net Net-(D1-A): track 6.62 -> 7.84 mm
- net Net-(R9-Pad2): track 6.60 -> 6.04 mm
Other:
- board size 50.3 x 66.3 mm -> 44.4 x 57.8 mm

Commit message: v3.0
Parts:
- Q1: footprint Package_TO_SOT_THT:TO-92_Inline -> Package_TO_SOT_THT:TO-92_Inline_Wide
- U1: footprint SensingStation:Z03A -> Package_TO_SOT_THT:TO-92_Inline
- moved R5 8.15 mm to (112.8, 91.8)
- moved R4 7.27 mm to (117.9, 105.1)
- moved U1 6.91 mm to (96.7, 110.0), turned to 90 degrees
- moved D2 6.40 mm to (99.4, 139.8), turned to 90 degrees
- moved R1 4.89 mm to (96.2, 104.5)
- moved R2 4.79 mm to (99.7, 104.4)
- moved C4 3.20 mm to (102.5, 132.5), turned to 0 degrees
- moved C2 3.18 mm to (92.7, 93.5)
- moved U3 3.08 mm to (85.2, 97.0)
- moved Q1 0.79 mm to (114.6, 96.8)
- moved R9 0.46 mm to (91.5, 114.7)
Routing:
- net +5V: track 92.8 -> 86.6 mm
- net /DAQ_LIGHT: track 24.0 -> 21.4 mm
- net Net-(U1-VO): track 4.07 -> 6.30 mm
- net /DAQ_SOUND: track 26.9 -> 24.7 mm
- net Net-(R4-Pad1): track 7.98 -> 6.17 mm
- net Net-(D1-A): track 7.84 -> 9.00 mm
- net Net-(U3B--): track 6.82 -> 7.92 mm
- net /DAQ_TEMP: track 14.9 -> 13.8 mm
- net Net-(D2-A): track 5.53 -> 4.96 mm
- net Net-(Q1-G): track 11.4 -> 11.9 mm
Other:
- board size 44.4 x 57.8 mm -> 42.7 x 57.8 mm

Commit message: version final
Parts:
- moved D2 0.76 mm to (99.2, 140.5)
Other:
- board size 42.7 x 57.8 mm -> 42.7 x 58.2 mm
Changed lines of the file:
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@@
 		(capping no)
 		(filling no)
-		(zone_defaults)
 		(pcbplotparams
 			(layerselection 0x00000000_00000000_55555555_5755f5ff)
@@
 	(footprint "LED_THT:LED_D5.0mm"
 		(layer "F.Cu")
-		(at 99.4 139.775 90)
+		(at 99.25 140.525 90)
 		(descr "LED, diameter 5.0mm, 2 pins, http://cdn-reichelt.de/documents/datenblatt/A500/LL-504BC2E-009.pdf, generated by kicad-footprint-generator")
 		(tags "LED")
@@
 		)
 		(point
-			(at 99.4 138.505)
+			(at 99.25 139.255)
 			(size 2)
 			(layer "F.Fab")
@@
 		(tags "LED")
 		(property "Reference" "D1"
-			(at 1.27 -3.96 90)
+			(at 3.76 -3.19 90)
 			(layer "F.SilkS")
 			(effects
@@
 		(tags "Resistor Axial_DIN0207 series Axial Horizontal pin pitch 10.16mm 0.25W = 1/4W length 6.3mm diameter 2.5mm")
 		(property "Reference" "R1"
-			(at -2.025 0.615 90)
+			(at 12.55 -0.05 90)
 			(layer "F.SilkS")
 			(effects
@@
 		(tags "Resistor Axial_DIN0207 series Axial Horizontal pin pitch 10.16mm 0.25W = 1/4W length 6.3mm diameter 2.5mm")
 		(property "Reference" "R2"
-			(at -2.275 0.415 90)
+			(at 12.45 -0.06 90)
 			(layer "F.SilkS")
 			(effects
@@
 		(tags "THT Terminal Block TE 282834-2 pitch 2.54mm size 5.54x6.5mm drill 1.1mm pad 2.1mm")
 		(property "Reference" "J2"
-			(at 0.37 -12.12 0)
+			(at -2.95 2.79 0)
 			(layer "F.SilkS")
 			(effects
@@
 		(tags "to-92 sc-43 sc-43a sot54 PA33 transistor")
 		(property "Reference" "Q1"
-			(at 2.54 -3.56 180)
+			(at -0.52 -3.46 180)
 			(layer "F.SilkS")
 			(effects
@@
 	(gr_rect
 		(start 78.85 87.55)
-		(end 121.5 145.35)
+		(end 121.5 145.75)
 		(stroke
 			(width 0.05)
@@
 		(layer "Edge.Cuts")
 	)
+	(dimension
+		(type aligned)
+		(layer "User.1")
+		(pts
+			(xy 79.13339 145.755912) (xy 79.324509 88.148632)
+		)
+		(height -10.824569)
+		(format
+			(prefix "")
+			(suffix "mm")
+			(units 3)
+			(units_format 0)
+			(precision 4)
+			(override_value "57.61")
+			(suppress_zeroes yes)
+		)
+		(style
+			(thickness 0.2)
+			(arrow_length 1.27)
+			(text_position_mode 0)
+			(arrow_direction outward)
+			(extension_height 0.58642)
+			(extension_offset 0.5)
+			(keep_text_aligned yes)
+		)
+		(gr_text "57.61mm"
+			(at 66.604451 116.910388 89.80991414)
+			(layer "User.1")
+			(effects
+				(font
+					(size 1.5 1.5)
+					(thickness 0.3)
+				)
+			)
+		)
+	)
+	(dimension
+		(type aligned)
+		(layer "User.1")
+		(pts
+			(xy 121.537846 88.025285) (xy 78.867846 88.005285)
+		)
+		(height 4.595286)
+		(format
+			(prefix "")
+			(suffix "mm")
+			(units 3)
+			(units_format 0)
+			(precision 4)
+			(suppress_zeroes yes)
+		)
+		(style
+			(thickness 0.2)
+			(arrow_length 1.27)
+			(text_position_mode 0)
+			(arrow_direction outward)
+			(extension_height 0.58642)
+			(extension_offset 0.5)
+			(keep_text_aligned yes)
+		)
+		(gr_text "42.67mm"
+			(at 100.205844 81.62 -0.02685529661)
+			(layer "User.1")
+			(effects
+				(font
+					(size 1.5 1.5)
+					(thickness 0.3)
+				)
+			)
+		)
+	)
 	(segment
-		(start 103.5 134.75)
-		(end 99.85 134.75)
+		(start 106.6 141.5)
+		(end 106.6 137.1)
 		(width 0.8)
 		(layer "B.Cu")
@@
 	)
 	(segment
-		(start 99.85 134.75)
+		(start 100.85 135.75)
 		(end 94.5 129.4)
 		(width 0.8)
@@
 	)
 	(segment
-		(start 94.5 129.4)
-		(end 94.5 126.925)
+		(start 106.6 137.1)
+		(end 105.25 135.75)
 		(width 0.8)
 		(layer "B.Cu")
@@
 	)
 	(segment
-		(start 97.415 126.925)
-		(end 97.445 126.895)
-		(width 0.4)
+		(start 94.5 129.4)
+		(end 94.5 126.925)
+		(width 0.8)
 		(layer "B.Cu")
 		(net "/DAQ_SOUND")
 	)
 	(segment
-		(start 106.6 137.85)
-		(end 103.5 134.75)
+		(start 105.25 135.75)
+		(end 100.85 135.75)
 		(width 0.8)
 		(layer "B.Cu")
@@
 	)
 	(segment
-		(start 106.6 141.5)
-		(end 106.6 137.85)
-		(width 0.8)
+		(start 97.415 126.925)
+		(end 97.445 126.895)
+		(width 0.4)
 		(layer "B.Cu")
 		(net "/DAQ_SOUND")
 	)
 	(segment
-		(start 94.65 137.235)
-		(end 94.5 137.085)
+		(start 99.25 137.985)
+		(end 95.4 137.985)
 		(width 0.8)
 		(layer "B.Cu")
@@
 	)
 	(segment
-		(start 99.4 137.235)
-		(end 94.65 137.235)
+		(start 95.4 137.985)
+		(end 94.5 137.085)
 		(width 0.8)
 		(layer "B.Cu")
@@
 	)
 	(segment
-		(start 103.45 91.9)
-		(end 102.02 91.9)
+		(start 117.95 136.38)
+		(end 114.73 136.38)
 		(width 0.8)
 		(layer "B.Cu")
-		(net "/DAQ_TEMP")
+		(net "/DAQ_MAG")
 	)
 	(segment
-		(start 102.02 91.9)
-		(end 99.7 94.22)
+		(start 114.73 136.38)
+		(end 114.6 136.51)
 		(width 0.8)
 		(layer "B.Cu")
-		(net "/DAQ_TEMP")
+		(net "/DAQ_MAG")
 	)
 	(segment
-		(start 94.39 99.53)
-		(end 99.7 94.22)
+		(start 114.6 136.51)
+		(end 114.13 136.51)
 		(width 0.8)
 		(layer "B.Cu")
-		(net "/DAQ_TEMP")
+		(net "/DAQ_MAG")
 	)
 	(segment
-		(start 92.815 99.53)
-		(end 94.39 99.53)
+		(start 114.13 136.51)
+		(end 109.14 141.5)
 		(width 0.8)
 		(layer "B.Cu")
-		(net "/DAQ_TEMP")
+		(net "/DAQ_MAG")
 	)
 	(segment
@@
 	)
 	(segment
-		(start 117.95 136.38)
-		(end 114.73 136.38)
+		(start 95.73 108.73)
+		(end 96.7 108.73)
 		(width 0.8)
 		(layer "B.Cu")
-		(net "/DAQ_MAG")
+		(net "Net-(U1-VO)")
 	)
 	(segment
-		(start 114.73 136.38)
-		(end 114.6 136.51)
+		(start 92.815 105.815)
+		(end 95.73 108.73)
 		(width 0.8)
 		(layer "B.Cu")
-		(net "/DAQ_MAG")
+		(net "Net-(U1-VO)")
 	)
 	(segment
-		(start 114.6 136.51)
-		(end 114.13 136.51)
+		(start 92.815 104.61)
+		(end 92.815 105.815)
 		(width 0.8)
 		(layer "B.Cu")
-		(net "/DAQ_MAG")
+		(net "Net-(U1-VO)")
 	)
 	(segment
-		(start 114.13 136.51)
-		(end 109.14 141.5)
+		(start 103.45 91.9)
+		(end 102.02 91.9)
 		(width 0.8)
 		(layer "B.Cu")
-		(net "/DAQ_MAG")
+		(net "/DAQ_TEMP")
 	)
 	(segment
-		(start 95.73 108.73)
-		(end 96.7 108.73)
+		(start 102.02 91.9)
+		(end 99.7 94.22)
 		(width 0.8)
 		(layer "B.Cu")
-		(net "Net-(U1-VO)")
+		(net "/DAQ_TEMP")
 	)
 	(segment
-		(start 92.815 105.815)
-		(end 95.73 108.73)
+		(start 94.39 99.53)
+		(end 99.7 94.22)
 		(width 0.8)
 		(layer "B.Cu")
-		(net "Net-(U1-VO)")
+		(net "/DAQ_TEMP")
 	)
 	(segment
-		(start 92.815 104.61)
-		(end 92.815 105.815)
+		(start 92.815 99.53)
+		(end 94.39 99.53)
 		(width 0.8)
 		(layer "B.Cu")
-		(net "Net-(U1-VO)")
+		(net "/DAQ_TEMP")
 	)
 	(zone
@@
 		(polygon
 			(pts
-				(xy 79.406498 87.872682) (xy 121.307423 87.752278) (xy 121.392609 144.869451) (xy 79.193496 144.8293)
+				(xy 78.999944 87.872682) (xy 121.30748 87.752278) (xy 121.393579 145.520118) (xy 79.191063 145.479962)
 			)
 		)
